File: Schematics/RenaultBT.kicad_pcb (KiCad board)
At the start: 2 copper layers, 160 x 100.3 mm, 62 parts, among them J1 PowerSupply, J2 SPDIF_Output, J3 HU_CDC_Interface, J4 Screw_Terminal_01x02, J5 Screw_Terminal_01x03, J6 Screw_Terminal_01x03, Q1 2N7000, Q2 2N7000, Q3 2N7000, Q4 2N7000, U1 LM2575-5.0BT, U2 LM3940, U3 WM8804, U4 CSRA64215, U5 74HC04, U6 STM32F103, Y1 12Mhz

Commit message: Minor fixes in PCB design
Parts:
- moved C4 1.27 mm to (128.3, 52.1)
- moved J1 1.27 mm to (203.2, 54.6)
- moved Q1 1.27 mm to (195.6, 62.2)
- moved R27 1.27 mm to (188.0, 57.1)
- moved U2 1.27 mm to (144.8, 52.1)
- moved C1 1.27 mm to (193.0, 47.0)
- moved C2 1.27 mm to (156.2, 58.4)
- moved D1 1.27 mm to (165.1, 47.0)
- moved J4 1.27 mm to (203.2, 73.7)
- moved J5 1.27 mm to (203.2, 86.4)
- moved J6 1.27 mm to (203.2, 101.6)
- moved L1 1.27 mm to (156.2, 47.0)
- moved R1 1.27 mm to (181.6, 61.0)
- moved R2 1.27 mm to (185.4, 47.0)
- moved U1 1.27 mm to (172.7, 47.0)
