File: Schematics/PowerSupply.sch (KiCad schematic (older format))
At the start: 11 parts, among them Q1 2N7000, U1 LM2575-5.0BT, U2 LM3940

Commit message: Fixed CDC interface schematic; Fixed SPDIF output interface schematic; Added screw terminals; Modified PCB design
Parts:
- Q1: footprint Package_TO_SOT_THT:TO-92_Inline -> Package_TO_SOT_THT:TO-92_Inline_Wide
Changed lines of the file:
@@
 F 0 "Q1" H 4555 4046 50  0000 L CNN
 F 1 "2N7000" H 4555 3955 50  0000 L CNN
-F 2 "Package_TO_SOT_THT:TO-92_Inline" H 4550 3925 50  0001 L CIN
+F 2 "Package_TO_SOT_THT:TO-92_Inline_Wide" H 4550 3925 50  0001 L CIN
 F 3 "https://www.fairchildsemi.com/datasheets/2N/2N7000.pdf" H 4350 4000 50  0001 L CNN
 F 4 "X" H 4350 4000 50  0001 C CNN "Spice_Primitive"
